File: controllers/original_pd-pi001.kicad_sch (KiCad schematic)
At the start: 47 parts, among them CN701 Cable, IC701 74HC157, IC702 74LS163, J701 Jumper_2_Bridged, J702 Jumper_2_Bridged, J703 Jumper_2_Bridged, J704 Jumper_2_Bridged, J705 Jumper_2_Bridged, J706 Jumper_2_Bridged, J707 Jumper_2_Bridged, J708 Jumper_2_Bridged, J709 Jumper_2_Bridged, J710 Jumper_2_Bridged, J711 Jumper_2_Bridged, J712 Jumper_2_Bridged, J713 Jumper_2_Bridged, J714 Jumper_2_Bridged, SW1 SWA, SW2 SWB, SW3 SWC, SW4 SWD, SW5 SWE, SW6 SWF, SW7 SWG, SW701 SW_SP3T, SW702 SW_SP3T, SW8 SWH

Commit message: upd
Parts:
- IC702: value 74LS163 -> 74HC163
- SW701: value SW_SP3T -> I_Turbo; footprint (none) -> PC_Engine:SW_Sliding_Surface_original
- SW702: value SW_SP3T -> II_Turbo; footprint (none) -> PC_Engine:SW_Sliding_Surface_original
Other:
- moved on the sheet: J703, J704, J705
Changed lines of the file:
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@@
 	)
 	(junction
-		(at 101.6 156.21)
+		(at 104.14 156.21)
 		(diameter 0)
 		(color 0 0 0 0)
@@
 	)
 	(junction
-		(at 111.76 153.67)
+		(at 114.3 153.67)
 		(diameter 0)
 		(color 0 0 0 0)
@@
 	)
 	(junction
-		(at 101.6 148.59)
+		(at 104.14 148.59)
 		(diameter 0)
 		(color 0 0 0 0)
 	)
 	(junction
-		(at 111.76 148.59)
+		(at 114.3 148.59)
 		(diameter 0)
 		(color 0 0 0 0)
@@
 	)
 	(junction
-		(at 101.6 153.67)
+		(at 104.14 153.67)
 		(diameter 0)
 		(color 0 0 0 0)
@@
 	)
 	(junction
-		(at 86.36 146.05)
+		(at 88.9 153.67)
 		(diameter 0)
 		(color 0 0 0 0)
@@
 	(wire
 		(pts
-			(xy 111.76 156.21) (xy 101.6 156.21)
+			(xy 114.3 156.21) (xy 104.14 156.21)
 		)
 		(stroke
@@
 	(wire
 		(pts
-			(xy 86.36 148.59) (xy 86.36 146.05)
+			(xy 88.9 156.21) (xy 88.9 153.67)
 		)
 		(stroke
@@
 	(wire
 		(pts
-			(xy 111.76 148.59) (xy 111.76 146.05)
+			(xy 114.3 148.59) (xy 114.3 146.05)
 		)
 		(stroke
@@
 	(wire
 		(pts
-			(xy 101.6 148.59) (xy 101.6 153.67)
+			(xy 104.14 148.59) (xy 104.14 153.67)
 		)
 		(stroke
@@
 	(wire
 		(pts
-			(xy 86.36 144.78) (xy 86.36 146.05)
+			(xy 88.9 152.4) (xy 88.9 153.67)
 		)
 		(stroke
@@
 	(wire
 		(pts
-			(xy 101.6 148.59) (xy 111.76 148.59)
+			(xy 104.14 148.59) (xy 114.3 148.59)
 		)
 		(stroke
@@
 	(wire
 		(pts
-			(xy 111.76 148.59) (xy 111.76 153.67)
+			(xy 114.3 148.59) (xy 114.3 153.67)
 		)
 		(stroke
@@
 	(wire
 		(pts
-			(xy 96.52 146.05) (xy 96.52 148.59)
+			(xy 99.06 153.67) (xy 99.06 156.21)
 		)
 		(stroke
@@
 	(wire
 		(pts
-			(xy 111.76 153.67) (xy 111.76 156.21)
+			(xy 114.3 153.67) (xy 114.3 156.21)
 		)
 		(stroke
@@
 	(wire
 		(pts
-			(xy 101.6 156.21) (xy 101.6 153.67)
+			(xy 104.14 156.21) (xy 104.14 153.67)
 		)
 		(stroke
@@
 	(wire
 		(pts
-			(xy 96.52 148.59) (xy 86.36 148.59)
+			(xy 99.06 156.21) (xy 88.9 156.21)
 		)
 		(stroke
@@
 	(wire
 		(pts
-			(xy 101.6 146.05) (xy 101.6 148.59)
+			(xy 104.14 146.05) (xy 104.14 148.59)
 		)
 		(stroke
@@
 	(wire
 		(pts
-			(xy 101.6 156.21) (xy 101.6 157.48)
+			(xy 104.14 156.21) (xy 104.14 157.48)
 		)
 		(stroke
@@
 	(symbol
 		(lib_id "Jumper:Jumper_2_Bridged")
-		(at 106.68 146.05 0)
+		(at 109.22 153.67 0)
 		(unit 1)
 		(body_style 1)
@@
 		(fields_autoplaced yes)
 		(property "Reference" "J705"
-			(at 106.68 143.51 0)
+			(at 109.22 151.13 0)
 			(show_name no)
 			(do_not_autoplace no)
@@
 		)
 		(property "Value" "Jumper_2_Bridged"
-			(at 106.68 140.97 0)
+			(at 109.22 148.59 0)
 			(hide yes)
 			(show_name no)
@@
 		)
 		(property "Footprint" "PC_Engine:Jumper_Controller_7.5mm"
-			(at 106.68 146.05 0)
+			(at 109.22 153.67 0)
 			(hide yes)
 			(show_name no)
@@
 		)
 		(property "Datasheet" ""
-			(at 106.68 151.13 0)
+			(at 109.22 158.75 0)
 			(hide yes)
 			(show_name no)
@@
 		)
 		(property "Description" "Jumper, 2-pole, closed/bridged"
-			(at 106.68 153.67 0)
+			(at 109.22 161.29 0)
 			(hide yes)
 			(show_name no)
@@
 			)
 		)
-		(property "Value" "SW_SP3T"
+		(property "Value" "II_Turbo"
 			(at 139.7 157.48 0)
 			(show_name no)
@@
 			)
 		)
-		(property "Footprint" ""
+		(property "Footprint" "PC_Engine:SW_Sliding_Surface_original"
 			(at 123.825 168.275 0)
 			(hide yes)
@@
 	(symbol
 		(lib_id "power:VCC")
-		(at 86.36 144.78 0)
+		(at 88.9 152.4 0)
 		(unit 1)
 		(body_style 1)
@@
 		(fields_autoplaced yes)
 		(property "Reference" "#PWR021"
-			(at 86.36 148.59 0)
+			(at 88.9 156.21 0)
 			(hide yes)
 			(show_name no)
@@
 		)
 		(property "Value" "VCC"
-			(at 86.36 139.7 0)
+			(at 88.9 147.32 0)
 			(show_name no)
 			(do_not_autoplace no)
@@
 		)
 		(property "Footprint" "Package_QFP:TQFP-44_10x10mm_P0.8mm"
-			(at 86.36 144.78 0)
+			(at 88.9 152.4 0)
 			(hide yes)
 			(show_name no)
@@
 		)
 		(property "Datasheet" ""
-			(at 86.36 144.78 0)
+			(at 88.9 152.4 0)
 			(hide yes)
 			(show_name no)
@@
 		)
 		(property "Description" "Power symbol creates a global label with name \"VCC\""
-			(at 86.36 144.78 0)
+			(at 88.9 152.4 0)
 			(hide yes)
 			(show_name no)
@@
 	(symbol
 		(lib_id "Jumper:Jumper_2_Bridged")
-		(at 91.44 146.05 0)
+		(at 93.98 153.67 0)
 		(unit 1)
 		(body_style 1)
@@
 		(fields_autoplaced yes)
 		(property "Reference" "J704"
-			(at 91.44 143.51 0)
+			(at 93.98 151.13 0)
 			(show_name no)
 			(do_not_autoplace no)
@@
 		)
 		(property "Value" "Jumper_2_Bridged"
-			(at 91.44 140.97 0)
+			(at 93.98 148.59 0)
 			(hide yes)
 			(show_name no)
@@
 		)
 		(property "Footprint" "PC_Engine:Jumper_Controller_7.5mm"
-			(at 91.44 146.05 0)
+			(at 93.98 153.67 0)
 			(hide yes)
 			(show_name no)
@@
 		)
 		(property "Datasheet" ""
-			(at 91.44 151.13 0)
+			(at 93.98 158.75 0)
 			(hide yes)
 			(show_name no)
@@
 		)
 		(property "Description" "Jumper, 2-pole, closed/bridged"
-			(at 91.44 153.67 0)
+			(at 93.98 161.29 0)
 			(hide yes)
 			(show_name no)
@@
 			)
 		)
-		(property "Value" "SW_SP3T"
+		(property "Value" "I_Turbo"
 			(at 139.7 140.97 0)
 			(show_name no)
@@
 			)
 		)
-		(property "Footprint" ""
+		(property "Footprint" "PC_Engine:SW_Sliding_Surface_original"
 			(at 123.825 151.765 0)
 			(hide yes)
@@
 	(symbol
 		(lib_id "power:GND")
-		(at 101.6 157.48 0)
+		(at 104.14 157.48 0)
 		(unit 1)
 		(body_style 1)
@@
 		(fields_autoplaced yes)
 		(property "Reference" "#PWR022"
-			(at 101.6 163.83 0)
+			(at 104.14 163.83 0)
 			(hide yes)
 			(show_name no)
@@
 		)
 		(property "Value" "GND"
-			(at 101.6 162.56 0)
+			(at 104.14 162.56 0)
 			(hide yes)
 			(show_name no)
@@
 		)
 		(property "Footprint" ""
-			(at 101.6 157.48 0)
+			(at 104.14 157.48 0)
 			(hide yes)
 			(show_name no)
@@
 		)
 		(property "Datasheet" ""
-			(at 101.6 157.48 0)
+			(at 104.14 157.48 0)
 			(hide yes)
 			(show_name no)
@@
 		)
 		(property "Description" "Power symbol creates a global label with name \"GND\" , ground"
-			(at 101.6 157.48 0)
+			(at 104.14 157.48 0)
 			(hide yes)
 			(show_name no)
@@
 			)
 		)
-		(property "Value" "74LS163"
+		(property "Value" "74HC163"
 			(at 159.6233 99.06 0)
 			(show_name no)
@@
 	(symbol
 		(lib_id "Jumper:Jumper_2_Bridged")
-		(at 106.68 153.67 0)
+		(at 109.22 146.05 0)
 		(unit 1)
 		(body_style 1)
@@
 		(fields_autoplaced yes)
 		(property "Reference" "J703"
-			(at 106.68 151.13 0)
+			(at 109.22 143.51 0)
 			(show_name no)
 			(do_not_autoplace no)
@@
 		)
 		(property "Value" "Jumper_2_Bridged"
-			(at 106.68 148.59 0)
+			(at 109.22 140.97 0)
 			(hide yes)
 			(show_name no)
@@
 		)
 		(property "Footprint" "PC_Engine:Jumper_Controller_7.5mm"
-			(at 106.68 153.67 0)
+			(at 109.22 146.05 0)
 			(hide yes)
 			(show_name no)
@@
 		)
 		(property "Datasheet" ""
-			(at 106.68 158.75 0)
+			(at 109.22 151.13 0)
 			(hide yes)
 			(show_name no)
@@
 		)
 		(property "Description" "Jumper, 2-pole, closed/bridged"
-			(at 106.68 161.29 0)
+			(at 109.22 153.67 0)
 			(hide yes)
 			(show_name no)
