File: controllers/original_pd-pi001.kicad_pcb (KiCad board)
At the start: 2 copper layers, 131 x 46.5 mm, 45 parts, among them CN701 Cable, IC701 74HC157, IC702 74LS163, J701 Jumper_2_Bridged, J702 Jumper_2_Bridged, J703 Jumper_2_Bridged, J704 Jumper_2_Bridged, J705 Jumper_2_Bridged, J706 Jumper_2_Bridged, J707 Jumper_2_Bridged, J708 Jumper_2_Bridged, J709 Jumper_2_Bridged, J710 Jumper_2_Bridged, J711 Jumper_2_Bridged, J712 Jumper_2_Bridged, J713 Jumper_2_Bridged, J714 Jumper_2_Bridged, SW1 SWA, SW2 SWB, SW3 SWC, SW4 SWD, SW5 SWE, SW6 SWF, SW7 SWG, SW8 SWH

Commit message: upd
Parts:
- added SW701: I_Turbo, PC_Engine:SW_Sliding_Surface_original, F.Cu at (197.1, 72.9)
- added SW702: II_Turbo, PC_Engine:SW_Sliding_Surface_original, F.Cu at (181.3, 72.9)
Routing:
- net Net-(R713-Pad2): track 24.8 -> 66.5 mm
- net Net-(R712-Pad1): track 14.1 -> 49.5 mm
- net Net-(R711-Pad2): track 23.6 -> 29.0 mm
Other:
- outline, holes or cut-outs redrawn

Commit message: fix
Routing:
- net Net-(IC701-I0a): track 93.7 -> 96.5 mm
